File: pcb/CJB.kicad_sch (KiCad schematic)
At the start: 38 parts, among them J1 USB_C_Receptacle_USB2.0_16P, Q1 BUK7880, SW1 SW_SPDT, U1 LM1117DT-3.3, U2 FT230XS, U3 INA181

Commit message: Change uart resistor values
Parts:
- R2, R4: value 1k -> 0; VendorId 102951 -> 102902
Changed lines of the file:
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@@
       (effects (font (size 1.27 1.27)))
     )
-    (property "Value" "1k" (at 134.62 45.72 90)
+    (property "Value" "0" (at 134.62 45.72 90)
       (effects (font (size 1.27 1.27)))
     )
@@
       (effects (font (size 1.27 1.27)) hide)
     )
-    (property "VendorId" "102951" (at 137.16 48.26 0)
+    (property "VendorId" "102902" (at 137.16 48.26 0)
       (effects (font (size 1.27 1.27)) hide)
     )
@@
       (effects (font (size 1.27 1.27)))
     )
-    (property "Value" "1k" (at 134.62 53.34 90)
+    (property "Value" "0" (at 134.62 53.34 90)
       (effects (font (size 1.27 1.27)))
     )
@@
       (effects (font (size 1.27 1.27)) hide)
     )
-    (property "VendorId" "102951" (at 137.16 50.8 0)
-      (effects (font (size 1.27 1.27)) hide)
-    )
+    (property "VendorId" "102902" (at 137.16 50.8 0)
+      (effects (font (size 1.27 1.27)) hide)
+    )
