File: pcb/CJB_audio.kicad_sch (KiCad schematic)
At the start: 35 parts, among them U5 PAM8406D, U6 PCM5100A

Commit message: Fix wrong vendor id
Parts:
- C12: VendorId 102598 -> 100135
Changed lines of the file:
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@@
       (effects (font (size 1.27 1.27)) hide)
     )
-    (property "VendorId" "102598" (at 173.99 74.93 0)
+    (property "VendorId" "100135" (at 173.99 74.93 0)
       (effects (font (size 1.27 1.27)) hide)
     )

Commit message: Fix boot and power issue
Connections:
- net +3V3: no longer C22.1, C23.2, U5.6 (VDD)
- net +5V: now also C22.1, C23.2, U5.6 (VDD)
Other:
- moved on the sheet: C22, C23, C24, C25, C26, C27

Commit message: Change SHDN and MUTE pins
Connections:
- net ~{MUTE}: now also U5.5 (~{MUTE}); no longer U5.12 (~{SHND})
- net ~{SHDN}: now also U5.12 (~{SHND}); no longer U5.5 (~{MUTE})
Changed lines of the file:
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@@
     )
   )
-  (global_label "~{SHDN}" (shape output) (at 134.62 77.47 0) (fields_autoplaced)
+  (global_label "~{SHDN}" (shape output) (at 134.62 74.93 0) (fields_autoplaced)
     (effects (font (size 1.27 1.27)) (justify left))
-    (property "Intersheetrefs" "${INTERSHEET_REFS}" (at 142.7457 77.47 0)
+    (property "Intersheetrefs" "${INTERSHEET_REFS}" (at 142.7457 74.93 0)
       (effects (font (size 1.27 1.27)) (justify left) hide)
     )
@@
     )
   )
-  (global_label "~{MUTE}" (shape output) (at 134.62 74.93 0) (fields_autoplaced)
+  (global_label "~{MUTE}" (shape output) (at 134.62 77.47 0) (fields_autoplaced)
     (effects (font (size 1.27 1.27)) (justify left))
-    (property "Intersheetrefs" "${INTERSHEET_REFS}" (at 142.5037 74.93 0)
+    (property "Intersheetrefs" "${INTERSHEET_REFS}" (at 142.5037 77.47 0)
       (effects (font (size 1.27 1.27)) (justify left) hide)
     )
