File: pcb/CJB.kicad_pcb (KiCad board)
At the start: 2 copper layers, 106.5 x 106.5 mm, 123 parts, among them J1 USB_C_Receptacle_USB2.0_16P, J2 Micro_SD_Card, J3 Conn_01x06_Socket, J4 Conn_01x06_Socket, J5 Conn_01x02_Pin, J6 Conn_01x02_Pin, J7 Conn_01x02_Pin, Q1 BUK7880, Q2 AO3400A, SW1 SW_SPDT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

Commit message: Rename apa102 spi clk/data pins
Connections:
- D4 pad 1: LED_SCK -> LED_DIN
- D4 pad 2: LED_DIN -> LED_SCK
- U4 pad 30: LED_SCK -> LED_DIN
- U4 pad 37: LED_DIN -> LED_SCK
Routing:
- net LED_SCK: track 42.8 -> 47.3 mm
- net LED_DIN: track 47.3 -> 42.8 mm
Changed lines of the file:
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@@
       (net 96 "unconnected-(U4-IO5-Pad29)") (pinfunction "IO5") (pintype "bidirectional+no_connect"))
     (pad "30" smd rect (at 8.75 1.905 180) (size 1.5 0.9) (layers "F.Cu" "F.Paste" "F.Mask")
-      (net 106 "LED_SCK") (pinfunction "IO18") (pintype "bidirectional"))
+      (net 16 "LED_DIN") (pinfunction "IO18") (pintype "bidirectional"))
     (pad "31" smd rect (at 8.75 0.635 180) (size 1.5 0.9) (layers "F.Cu" "F.Paste" "F.Mask")
       (net 97 "unconnected-(U4-IO19-Pad31)") (pinfunction "IO19") (pintype "bidirectional+no_connect"))
@@
       (net 88 "AUDIO_DATA") (pinfunction "IO22") (pintype "bidirectional"))
     (pad "37" smd rect (at 8.75 -6.985 180) (size 1.5 0.9) (layers "F.Cu" "F.Paste" "F.Mask")
-      (net 16 "LED_DIN") (pinfunction "IO23") (pintype "bidirectional"))
+      (net 106 "LED_SCK") (pinfunction "IO23") (pintype "bidirectional"))
     (pad "38" smd rect (at 8.75 -8.255 180) (size 1.5 0.9) (layers "F.Cu" "F.Paste" "F.Mask")
       (net 2 "GND") (pinfunction "GND") (pintype "passive"))
@@
       (stroke (width 0.1) (type solid)) (fill none) (layer "F.Fab"))
     (pad "1" smd rect (at -2.4 -1.7 90) (size 1.1 2) (layers "F.Cu" "F.Paste" "F.Mask")
-      (net 106 "LED_SCK") (pinfunction "DI") (pintype "input"))
+      (net 16 "LED_DIN") (pinfunction "DI") (pintype "input"))
     (pad "2" smd rect (at -2.4 0 90) (size 1.1 2) (layers "F.Cu" "F.Paste" "F.Mask")
-      (net 16 "LED_DIN") (pinfunction "CI") (pintype "input"))
+      (net 106 "LED_SCK") (pinfunction "CI") (pintype "input"))
     (pad "3" smd rect (at -2.4 1.7 90) (size 1.1 2) (layers "F.Cu" "F.Paste" "F.Mask")
       (net 2 "GND") (pinfunction "GND") (pintype "power_in"))
@@
   (via (at 135.89 72.85) (size 0.4) (drill 0.3) (layers "F.Cu" "B.Cu") (net 15))
   (segment (start 135.89 72.85) (end 135.89 94.8632) (width 0.4) (layer "B.Cu") (net 15))
-  (segment (start 135.382 46.355) (end 137.122 44.615) (width 0.4) (layer "F.Cu") (net 16))
-  (segment (start 137.122 44.615) (end 141.11 44.615) (width 0.4) (layer "F.Cu") (net 16))
-  (segment (start 130.95 83.01) (end 129.286 83.01) (width 0.4) (layer "F.Cu") (net 16))
-  (via (at 129.286 83.01) (size 0.4) (drill 0.3) (layers "F.Cu" "B.Cu") (net 16))
-  (via (at 135.382 46.355) (size 0.4) (drill 0.3) (layers "F.Cu" "B.Cu") (net 16))
-  (segment (start 135.382 52.324) (end 129.286 58.42) (width 0.4) (layer "B.Cu") (net 16))
-  (segment (start 129.286 58.42) (end 129.286 83.01) (width 0.4) (layer "B.Cu") (net 16))
-  (segment (start 135.382 46.355) (end 135.382 52.324) (width 0.4) (layer "B.Cu") (net 16))
+  (segment (start 136.282 42.915) (end 141.11 42.915) (width 0.4) (layer "F.Cu") (net 16))
+  (segment (start 133.858 45.339) (end 136.282 42.915) (width 0.4) (layer "F.Cu") (net 16))
+  (segment (start 127.762 74.12) (end 130.95 74.12) (width 0.4) (layer "F.Cu") (net 16))
+  (via (at 133.858 45.339) (size 0.4) (drill 0.3) (layers "F.Cu" "B.Cu") (net 16))
+  (via (at 127.762 74.12) (size 0.4) (drill 0.3) (layers "F.Cu" "B.Cu") (net 16))
+  (segment (start 127.762 57.658) (end 127.762 74.12) (width 0.4) (layer "B.Cu") (net 16))
+  (segment (start 133.858 51.562) (end 127.762 57.658) (width 0.4) (layer "B.Cu") (net 16))
+  (segment (start 133.858 45.339) (end 133.858 51.562) (width 0.4) (layer "B.Cu") (net 16))
   (arc (start 145.923 44.577001) (mid 156.492573 46.230326) (end 166.470086 50.090193) (width 0.4) (layer "F.Cu") (net 17))
   (arc (start 145.923 42.926) (mid 156.982123 44.654243) (end 167.410848 48.720287) (width 0.4) (layer "F.Cu") (net 18))
@@
   (via (at 147.5287 94.2132) (size 0.4) (drill 0.3) (layers "F.Cu" "B.Cu") (net 105))
   (segment (start 147.5287 92.71) (end 147.5287 94.2132) (width 0.4) (layer "B.Cu") (net 105))
-  (segment (start 136.282 42.915) (end 141.11 42.915) (width 0.4) (layer "F.Cu") (net 106))
-  (segment (start 133.858 45.339) (end 136.282 42.915) (width 0.4) (layer "F.Cu") (net 106))
-  (segment (start 127.762 74.12) (end 130.95 74.12) (width 0.4) (layer "F.Cu") (net 106))
-  (via (at 133.858 45.339) (size 0.4) (drill 0.3) (layers "F.Cu" "B.Cu") (net 106))
-  (via (at 127.762 74.12) (size 0.4) (drill 0.3) (layers "F.Cu" "B.Cu") (net 106))
-  (segment (start 127.762 57.658) (end 127.762 74.12) (width 0.4) (layer "B.Cu") (net 106))
-  (segment (start 133.858 51.562) (end 127.762 57.658) (width 0.4) (layer "B.Cu") (net 106))
-  (segment (start 133.858 45.339) (end 133.858 51.562) (width 0.4) (layer "B.Cu") (net 106))
+  (segment (start 135.382 46.355) (end 137.122 44.615) (width 0.4) (layer "F.Cu") (net 106))
+  (segment (start 137.122 44.615) (end 141.11 44.615) (width 0.4) (layer "F.Cu") (net 106))
+  (segment (start 130.95 83.01) (end 129.286 83.01) (width 0.4) (layer "F.Cu") (net 106))
+  (via (at 129.286 83.01) (size 0.4) (drill 0.3) (layers "F.Cu" "B.Cu") (net 106))
+  (via (at 135.382 46.355) (size 0.4) (drill 0.3) (layers "F.Cu" "B.Cu") (net 106))
+  (segment (start 135.382 52.324) (end 129.286 58.42) (width 0.4) (layer "B.Cu") (net 106))
+  (segment (start 129.286 58.42) (end 129.286 83.01) (width 0.4) (layer "B.Cu") (net 106))
+  (segment (start 135.382 46.355) (end 135.382 52.324) (width 0.4) (layer "B.Cu") (net 106))
   (segment (start 133.35 85.471) (end 139.954 85.471) (width 0.4) (layer "F.Cu") (net 107))
   (via (at 133.35 85.471) (size 0.4) (drill 0.3) (layers "F.Cu" "B.Cu") (net 107))
